Commit message: Release v0.2.1: T1-T5 product cells including thin ros2 Dual.
URDF contact extract, desk stand log, soils workbench, and ha-dual-ros2 / ament package so robot_description inserts Dual without a Gazebo stack. Badge dual+ros2; CI smoke for T5.

Co-authored-by: Cursor <cursoragent@cursor.com>

File: fixtures/open_registry/urdf/ros_skidsteer_v1.urdf (robot description, URDF)
Before this commit: robot ros_skidsteer_v1, 4 links, 3 joints
Links:
- link base_link: mass None -> 50.0; geometry collision box size=0.4 0.28 0.12; visual box size=0.4 0.28 0.12
- link track_left_link: mass None -> 6.0; geometry collision cylinder length=0.28 radius=0.06; visual cylinder length=0.28 radius=0.06
- link track_right_link: mass None -> 6.0; geometry collision cylinder length=0.28 radius=0.06; visual cylinder length=0.28 radius=0.06
